File: Simple/SimplePiddy.brd (EAGLE design)
At the start: 47.9 x 75 mm, 19 parts

Commit message: Lots of Updates
Created second Simple Piddy.
Updates to Complex Piddy
Parts:
- BT1, BT2: device microbuilder:JSTSH2 -> microbuilder:JSTPH2STRAIGHT
- moved BT2 6.30 mm to (3.75, 26.3)
- moved BT1 3.16 mm to (3.81, 35.0)
- moved POWER 1.60 mm to (8.60, 72.0)
- moved MOTORS 1.50 mm to (8.00, 62.5)
Connections:
- net GND: now also BT2.2; no longer BT1.1
- net N$18: now also BT1.1; no longer BT2.2
Routing:
- net N$18: track 45.0 -> 40.5 mm
- net N$17: track 5.44 -> 8.15 mm
- net RAW: track 37.0 -> 35.6 mm
- net N$1: track 62.5 -> 61.9 mm
Other:
- board text added: "BT1"
- board text added: "BT2"
- board text added: "MOTORS"
- board text added: "MTA"
- board text added: "MTB"
- board text added: "P"
- board text added: "POWER"
- board text added: "S1"
