File: Board_V1/PIDDYBOT_V1.brd (EAGLE design)
At the start: 48 x 76 mm, 76 parts, among them IC1 FT232RLSSOP, IC2 LMV358, IC3 LM1117, Q1 MOSFET-PCHANNELSMD, Q2 MOSFET-NCHANNELSMD, Q3 MOSFET-NCHANNELSMD, U1 MPU-6050-1, U2 MIC5205, U3 ATMEGA328, U4 TB6621FNG, U5 BLUETOOTH-RN41, Y1 16MHz

Commit message: Lots of Updates
Created second Simple Piddy.
Updates to Complex Piddy
Parts:
- removed C10, C12: 0.1uF, SparkFun:0402-CAP
- removed C11: 0.1uF, SparkFun-Capacitors:0402-CAP
- removed C15: 10uF, SparkFun-Capacitors:EIA3216
- removed C3: 10uF, SparkFun:EIA3216
- removed D1: MBRA140, SparkFun:SMA-DIODE
- removed F1: 500mA, SparkFun:PTC-1206
- removed IC1: FT232RLSSOP, SparkFun-DigitalIC:SSOP28DB
- removed IC3: LM1117, Testing:SOT223-ALT1
- removed LED3: RED, SparkFun:LED-0603
- removed LED4: YELLOW, SparkFun:LED-0603
- removed R14: 715, SparkFun:0402-RES
- removed R15: 240, SparkFun:0402-RES
- removed R6, R7, R8, R9: 1k, SparkFun:0402-RES
- removed U$13: USB-MINIB-5PIN, SparkFun-Connectors:USB-MINIB
- added IC7: TLV71333DBV, anoven:SOT-23-5
- C1: value 0.1uF -> 100nF; device SparkFun:0402-CAP -> rcl:C0603K
- C2: value 47uF -> 100nF; device SparkFun:PANASONIC_D -> rcl:C0603K
- moved C1 50.3 mm to (-2.00, -17.0), turned to 0 degrees
- moved R10 26.8 mm to (24.0, 55.0)
- moved C16 25.0 mm to (19.5, 53.5)
- moved SJ3 24.6 mm to (23.0, 54.0)
- moved R18 22.5 mm to (54.5, 28.0)
- moved SJ2 22.4 mm to (29.0, 54.5)
- moved C9 22.0 mm to (23.5, 51.5)
- moved R3 20.8 mm to (4.50, 55.5)
- moved R16 20.6 mm to (57.5, 25.0)
- moved C14 20.1 mm to (21.0, 58.0)
- moved C2 19.4 mm to (3.00, 44.0), turned to 0 degrees
- moved U1 19.0 mm to (30.0, 53.0)
- moved Q2 18.2 mm to (54.0, 24.0)
- moved S1 15.8 mm to (12.5, 57.0), turned to 270 degrees
- moved R19 14.9 mm to (56.5, 19.0)
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Connections:
- removed net D+: IC1.15, U$13.D+
- removed net D-: IC1.16, U$13.D-
- removed net N$10: LED4.A, R7.2
- removed net N$12: CN1.2, CN2.1
- removed net N$13: CN2.2, S3.1
- removed net N$15: IC3.1, R14.2, R15.1
- removed net RXD: IC1.5, R9.2
- removed net RXLED: IC1.22, LED4.C
- removed net TXD: IC1.1, R8.2
- removed net TXLED: IC1.23, LED3.C
- removed net VIN1: C2.+, D1.C, IC3.3
- removed net VUSB: C10.1, F1.1, U$13.VBUS
- new net VBATT: C2.1, IC7.1, IC7.3
- new net VCC: C1.1, IC7.5
- new net V_BATT: S3.3
- net 5V: no longer C1.1, C11.1, C15.A, C3.A, IC1.20, IC1.4, IC3.2, IC3.4, R15.2, R6.1, R7.1
- net DTR: no longer IC1.2
- net GND: now also C2.2, CN2.1, IC7.2; no longer C10.2, C11.2, C12.2, C15.C, C2.-, C3.C, CN1.1, IC1.18, IC1.21, IC1.25, IC1.26, IC1.7, R14.1, U$13.GND, U$13.MTN1, U$13.MTN2, U$13.MTN3, U$13.MTN4
- net N$1: now also S3.2; no longer C12.1, IC1.17
- net N$8: now also CN1.1, CN2.2; no longer LED3.A, R6.2
- net PWRIN: no longer D1.A, S3.2
- net RX-I: no longer R8.1
- net TX-O: no longer R9.1
- net USBVCC: no longer F1.2
Routing:
- removed copper zone on layer 1, net GND
- removed copper zone on layer 16, net GND

Commit message: initial commit
Parts:
- removed C7: 1uF, SparkFun:0402-CAP
- removed IC2: LMV358, SparkFun:SO08
- removed LED2: GREEN, SparkFun:LED-0603
- removed Q1: MOSFET-PCHANNELSMD, SparkFun:SOT23-3
- removed Q2, Q3: MOSFET-NCHANNELSMD, SparkFun:SOT23-3
- removed R13, R16, R17, R18, R19, R20: 10K, SparkFun:0402-RES
- removed R5: 10k, SparkFun:0402-RES
- removed SJ2, SJ3: (no value), SparkFun:SJ_2S-TRACE
- removed SJ4: SOLDERJUMPERNO, SparkFun:SJ_2S-NO
- added C3: 4.7uF, SparkFun:0402-CAP
- added D1: (no value), SparkFun-DiscreteSemi:SOD-323
- added D11: RED, SparkFun:LED-0603
- added JP1: (no value), SparkFun-Connectors:1X06-SMD
- added U$2, U$3: AYZ0202, SparkFun-Electromechanical:AYZ0202
- added X1: Micro USB, SparkFun:USB-MINIB
- C6: value 0.1uF -> 4.7uF
- CN1, CN2: value (none) -> M02JST-PTH-2; device microbuilder:JSTSH2 -> SparkFun-Connectors:JST-2-PTH
- R2: value 1k -> 330
- R4: value 10k -> 2K
- U2: value MIC5205 -> MCP73831
- Y1: value 16MHz -> 8Mhz; device SparkFun-FreqCtrl:RESONATOR-SMD -> murata-filter:CSTCR6M
- moved C1 69.4 mm to (8.50, 51.6), turned to 180 degrees
- moved R4 54.7 mm to (6.12, 73.1)
- moved U2 49.7 mm to (8.50, 68.4), turned to 0 degrees
- moved C6 46.9 mm to (10.1, 65.4), turned to 0 degrees
- moved JP2 39.7 mm to (46.0, 62.0)
- moved LED1 39.5 mm to (28.7, 26.9), turned to 180 degrees
- moved R22 39.5 mm to (46.0, 65.4), turned to 270 degrees
- moved R2 39.4 mm to (8.88, 74.8)
- moved R1 38.6 mm to (28.6, 30.0), turned to 270 degrees
- moved C8 20.4 mm to (19.4, 45.0)
- moved C13 18.6 mm to (23.9, 45.5), turned to 0 degrees
- moved C17 13.8 mm to (18.0, 19.2), turned to 180 degrees
- moved Y1 11.5 mm to (17.5, 30.5), turned to 0 degrees
- moved C4 11.3 mm to (30.0, 37.9)
- moved C18 10.6 mm to (24.5, 25.2)
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Connections:
- removed net 3.3V: C7.1, IC2.2, Q2.1, Q3.1, R13.1, R18.1, U2.5, U5.11
- removed net 3V3: C14.1, R10.2, R11.2, SJ1.1, U1.13
- removed net 5V: C18.1, C5.2, C6.1, IC2.8, Q1.2, R16.1, R19.1, R2.2, R3.2, U$16.P$3, U$17.P$3, U$18.P$3, U2.1, U2.3, U3.18, U3.4, U3.6, U4.20
- removed net CLKIN: SJ2.2, U1.1
- removed net CMP: IC2.3, R4.1, R5.2
- removed net CTS_5V: R17.2
- removed net FSYNC: SJ3.2, U1.11
- removed net GATE_CMD: IC2.1, Q1.1
- removed net IO6: U3.10
- removed net PWRIN: C17.1, C19.A, U4.13, U4.14, U4.24
- removed net RTS_5V: Q2.3, R16.2
- removed net RXBT: R20.1, U5.13
- removed net RX_5V: R20.2
- removed net TXBT: Q3.2, R18.2, U5.14
- removed net TX_5V: Q3.3, R19.2
- removed net USBVCC: Q1.3
- removed net VBATT: C2.1, IC7.1, IC7.3
- new net BT-RXI: U$3.3, U5.13
- new net BT-TXO: U$3.6, U5.14
- new net CHARGE: CN2.2, D1.1, S3.2, U$2.4
- new net N$10: U$2.3, U$2.6
- new net N$13: D11.A, R2.1
- new net PROG: R4.1, U2.5
- new net PROG-RXI: JP1.2, U$3.4
- new net PROG-TXO: JP1.3, U$3.1
- new net STAT: D11.C, U2.1
- net CTS: no longer R17.1, SJ4.2
- net DTR: now also JP1.1
- net GND: now also C3.2, CN1.1, JP1.6, R4.2, U$2.1, X1.GND; no longer C7.2, CN2.1, IC2.4, IC2.5, IC2.6, LED2.C, R5.1, SJ2.1, SJ3.1
- net N$1: now also C6.1, D1.2, U2.3; no longer S3.2
- net N$2: now also CN2.1, U$2.2; no longer LED2.A, R2.1
- net N$8: now also CN1.2, U$2.5; no longer CN1.1, CN2.2
- net PWMA: now also U3.10; no longer U3.1
- net RTS: no longer Q2.2, R13.2, SJ4.1
- net RX-I: now also U$3.5
- net TX-O: now also U$3.2
- net VCC: now also C14.1, C18.1, C5.2, JP1.4, R10.2, R11.2, R3.2, SJ1.1, U$16.P$3, U$17.P$3, U$18.P$3, U1.13, U3.18, U3.4, U3.6, U4.20, U5.11
- net VIN: now also C3.1, R2.2, U2.4, X1.VBUS; no longer R4.2
- net V_BATT: now also C17.1, C19.A, C2.1, IC7.1, IC7.3, U4.13, U4.14, U4.24
Routing:
- net VCC: track 0.00 -> 158.3 mm, vias 0 -> 3
- net V_BATT: track 0.00 -> 70.0 mm
- net DTR: track 0.00 -> 41.0 mm, vias 0 -> 1
- net POTD: track 0.00 -> 40.1 mm, vias 0 -> 1
- net CHARGE: track 0.00 -> 39.2 mm
- net RX-I: track 0.00 -> 30.3 mm, vias 0 -> 1
- net RESET: track 0.00 -> 29.3 mm, vias 0 -> 2
- net POTP: track 0.00 -> 29.3 mm
- net BT-RXI: track 0.00 -> 26.3 mm, vias 0 -> 1
- net N$11: track 0.00 -> 25.1 mm
- net PIO4: track 0.00 -> 25.1 mm
- net POTI: track 0.00 -> 24.8 mm, vias 0 -> 1
- net VIN: track 0.00 -> 23.8 mm
- net TX-O: track 0.00 -> 22.9 mm, vias 0 -> 1
- net PWMB: track 0.00 -> 19.9 mm, vias 0 -> 2
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- added copper zone on layer 1, net GND
- added copper zone on layer 16, net GND
Other:
- board text added: "M-OFF"
- board text added: "M-ON"

Commit message: Latest PIDDYBOT pcb finished ready to order
Parts:
- removed D1: (no value), SparkFun-DiscreteSemi:SOD-323
- added D4: (no value), microbuilder:SOT23-R
Connections:
- net CHARGE: now also D4.3; no longer D1.1
- net N$1: now also D4.1, D4.2; no longer D1.2
Routing:
- net N$1: track 4.54 -> 9.07 mm
- net CHARGE: track 39.2 -> 37.7 mm
- net STAT: track 5.43 -> 4.86 mm
Changed lines of the file:
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@@
 </element>
 <element name="JP1" library="SparkFun-Connectors" package="1X06-SMD" value="" x="40.625" y="39" smashed="yes" rot="MR270"/>
-<element name="D1" library="SparkFun-DiscreteSemi" package="SOD-323" value="" x="5.5" y="65.375" smashed="yes">
-<attribute name="PROD_ID" value="DIO-09646" x="5.5" y="65.375" size="1.778" layer="27" display="off"/>
-<attribute name="NAME" x="3.736" y="66.391" size="0.8128" layer="25"/>
-<attribute name="VALUE" x="4.484" y="63.978" size="0.4064" layer="27"/>
-</element>
+<element name="D4" library="microbuilder" package="SOT23-R" value="" x="3.375" y="65.125" rot="R180"/>
 </elements>
 <signals>
@@
 <contactref element="D11" pad="C"/>
 <contactref element="U2" pad="1"/>
-<wire x1="7.55" y1="67.0749" x2="7.5" y2="67.1249" width="0.2" layer="1"/>
-<wire x1="7.5" y1="67.1249" x2="7.5" y2="68.5" width="0.2" layer="1"/>
-<wire x1="7.5" y1="68.5" x2="7.75" y2="68.75" width="0.2" layer="1"/>
-<wire x1="7.75" y1="68.75" x2="8.375" y2="68.75" width="0.2" layer="1"/>
-<wire x1="8.375" y1="68.75" x2="8.75" y2="69.125" width="0.2" layer="1"/>
-<wire x1="8.75" y1="69.125" x2="8.75" y2="70.25" width="0.2" layer="1"/>
-<wire x1="8.75" y1="70.25" x2="8.5" y2="70.5" width="0.2" layer="1"/>
-<wire x1="8.5" y1="70.5" x2="8.5" y2="71.5" width="0.2" layer="1"/>
+<wire x1="7.55" y1="67.0749" x2="7.625" y2="67.0749" width="0.3048" layer="1"/>
+<wire x1="7.625" y1="67.0749" x2="7.625" y2="68.125" width="0.3048" layer="1"/>
+<wire x1="7.625" y1="68.125" x2="8.5" y2="69" width="0.3048" layer="1"/>
+<wire x1="8.5" y1="69" x2="8.5" y2="71.5" width="0.3048" layer="1"/>
 </signal>
 <signal name="CHARGE">
@@
 <wire x1="2.25" y1="54" x2="1" y2="55.25" width="0.6096" layer="1"/>
 <wire x1="1" y1="55.25" x2="1" y2="62.625" width="0.6096" layer="1"/>
-<wire x1="1" y1="62.625" x2="3.75" y2="65.375" width="0.6096" layer="1"/>
-<contactref element="D1" pad="1"/>
-<wire x1="3.75" y1="65.375" x2="4.35" y2="65.375" width="0.6096" layer="1"/>
+<contactref element="D4" pad="3"/>
+<wire x1="1" y1="62.625" x2="2.5" y2="64.125" width="0.6096" layer="1"/>
+<wire x1="2.5" y1="64.125" x2="3.375" y2="64.125" width="0.6096" layer="1"/>
 </signal>
 <signal name="BT-TXO">
@@
 <wire x1="9.45" y1="67.0749" x2="9.475" y2="67.0499" width="0.4064" layer="1"/>
 <wire x1="9.475" y1="67.0499" x2="9.475" y2="65.375" width="0.4064" layer="1"/>
-<contactref element="D1" pad="2"/>
-<wire x1="6.65" y1="65.375" x2="9.475" y2="65.375" width="0.6096" layer="1"/>
+<contactref element="D4" pad="2"/>
+<contactref element="D4" pad="1"/>
+<wire x1="9.475" y1="65.375" x2="5.075" y2="65.375" width="0.6096" layer="1"/>
+<wire x1="5.075" y1="65.375" x2="4.325" y2="66.125" width="0.6096" layer="1"/>
+<wire x1="4.325" y1="66.125" x2="2.425" y2="66.125" width="0.6096" layer="1"/>
 </signal>
 </signals>
