File: Board_V1/PIDDYBOT_V1.sch (EAGLE design)
At the start: 76 parts, among them IC1 FT232RLSSOP, IC2 LMV358, IC3 LM1117, Q1 MOSFET-PCHANNELSMD, Q2 MOSFET-NCHANNELSMD, Q3 MOSFET-NCHANNELSMD, U1 MPU-6050-1, U2 MIC5205, U3 ATMEGA328, U4 TB6621FNG, U5 BLUETOOTH-RN41, Y1 16MHz

Commit message: Lots of Updates
Created second Simple Piddy.
Updates to Complex Piddy
Parts:
- removed C10, C12: 0.1uF, SparkFun:CAP0402-CAP
- removed C11: 0.1uF, SparkFun-Capacitors:CAP0402-CAP
- removed C15: 10uF, SparkFun-Capacitors:CAP_POL1206
- removed C3: 10uF, SparkFun:CAP_POL1206
- removed D1: MBRA140, SparkFun:DIODE-SCHOTTKY_
- removed F1: 500mA, SparkFun:PTCSMD
- removed IC1: FT232RLSSOP, SparkFun-DigitalIC:FT232RLSSOP
- removed IC3: LM1117, Testing:V_REG_LM1117ALT1
- removed LED3: RED, SparkFun:LED0603
- removed LED4: YELLOW, SparkFun:LED0603
- removed R14: 715, SparkFun:RESISTOR0402-RES
- removed R15: 240, SparkFun:RESISTOR0402-RES
- removed R6, R7, R8, R9: 1k, SparkFun:RESISTOR0402-RES
- removed U$13: USB-MINIB-5PIN, SparkFun-Connectors:USB-MINIB-5PIN
- added IC7: TLV71333DBV, anoven:TLV71333DBV
- C1: value 0.1uF -> 100nF; device SparkFun:CAP0402-CAP -> rcl:C-EUC0603K
- C2: value 47uF -> 100nF; device SparkFun:CAP_POLD -> rcl:C-EUC0603K
Connections:
- removed net D+: IC1.USBDP, U$13.D+
- removed net D-: IC1.USBDM, U$13.D-
- removed net N$10: LED4.A, R7.2
- removed net N$12: CN1.2, CN2.1
- removed net N$13: CN2.2, S3.O
- removed net N$15: IC3.ADJ, R14.2, R15.1
- removed net RXD: IC1.RXD, R9.2
- removed net RXLED: IC1.RXLED, LED4.C
- removed net TXD: IC1.TXD, R8.2
- removed net TXLED: IC1.TXLED, LED3.C
- removed net VIN1: C2.+, D1.C, IC3.IN
- removed net VUSB: C10.1, F1.1, U$13.VBUS
- new net VBATT: C2.1, IC7.EN, IC7.IN
- new net VCC: C1.1, IC7.OUT
- new net V_BATT: S3.S
- net 5V: no longer C1.1, C11.1, C15.+, C3.+, IC1.VCC, IC1.VCCIO, IC3.OUT, IC3.OUT@1, R15.2, R6.1, R7.1
- net DTR: no longer IC1.DTR
- net GND: now also C2.2, CN2.1, IC7.GND; no longer C10.2, C11.2, C12.2, C15.-, C2.-, C3.-, CN1.1, IC1.AGND, IC1.GND18, IC1.GND21, IC1.GND7, IC1.TEST, R14.1, U$13.GND, U$13.MTN1, U$13.MTN2, U$13.MTN3, U$13.MTN4
- net N$1: now also S3.P; no longer C12.1, IC1.3V3OUT
- net N$8: now also CN1.1, CN2.2; no longer LED3.A, R6.2
- net PWRIN: no longer D1.A, S3.P
- net RX-I: no longer R8.1
- net TX-O: no longer R9.1
- net USBVCC: no longer F1.2
Other:
- note added: "3v3 Reg"
- note removed: "FT232RL (USB-to-Serial Converter)"
- note removed: "Vin / 5V Regulator"
- moved on the sheet: C1, CN1, CN2, Q2, Q3, R13, R16, R17, R18, R19, R20, S3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

Commit message: initial commit
Parts:
- removed C7: 1uF, SparkFun:CAP0402-CAP
- removed IC2: LMV358, SparkFun:OPAMP-DUALU
- removed LED2: GREEN, SparkFun:LED0603
- removed Q1: MOSFET-PCHANNELSMD, SparkFun:MOSFET-PCHANNELSMD
- removed Q2, Q3: MOSFET-NCHANNELSMD, SparkFun:MOSFET-NCHANNELSMD
- removed R13, R16, R17, R18, R19, R20: 10K, SparkFun:RESISTOR0402-RES
- removed R5: 10k, SparkFun:RESISTOR0402-RES
- removed SJ2, SJ3: SOLDERJUMPERTRACE, SparkFun:SOLDERJUMPERTRACE
- removed SJ4: SOLDERJUMPERNO, SparkFun:SOLDERJUMPERNO
- added C3: 4.7uF, SparkFun:CAP0402-CAP
- added D1: (no value), SparkFun-DiscreteSemi:DIODESOD
- added D11: RED, SparkFun:LED0603
- added JP1: (no value), SparkFun-Connectors:ARDUINO_SERIAL_PROGRAMSMD
- added U$2, U$3: AYZ0202, SparkFun-Electromechanical:AYZ0202
- added X1: Micro USB, SparkFun:USBSMD
- C6: value 0.1uF -> 4.7uF
- CN1, CN2: value (none) -> M02JST-PTH-2; device microbuilder:JST_2PINSH2 -> SparkFun-Connectors:M02JST-PTH-2
- R2: value 1k -> 330
- R4: value 10k -> 2K
- U2: value MIC5205 -> MCP73831; device SparkFun:V_REG_LDOSMD -> SparkFun:MCP73831
- Y1: value 16MHz -> 8Mhz; device SparkFun-FreqCtrl:RESONATORSMD -> murata-filter:CSTCR6M00G53Z
Connections:
- removed net 3.3V: C7.1, IC2A.-IN, Q2.G, Q3.G, R13.1, R18.1, U2.OUT, U5.VDD
- removed net 3V3: C14.1, R10.2, R11.2, SJ1.1, U1.VDD
- removed net 5V: C18.1, C5.2, C6.1, IC2A.V+, Q1.S, R16.1, R19.1, R2.2, R3.2, U$16.A, U$17.A, U$18.A, U2.EN, U2.IN, U3.AVCC, U3.VCC@1, U3.VCC@2, U4.VCC
- removed net CLKIN: SJ2.2, U1.CLKIN
- removed net CMP: IC2A.+IN, R4.1, R5.2
- removed net CTS_5V: R17.2
- removed net FSYNC: SJ3.2, U1.FSYNC
- removed net GATE_CMD: IC2A.OUT, Q1.G
- removed net IO6: U3.PD6(AIN0)
- removed net PWRIN: C17.1, C19.+, U4.VM1, U4.VM2, U4.VM3
- removed net RTS_5V: Q2.D, R16.2
- removed net RXBT: R20.1, U5.UARTRX
- removed net RX_5V: R20.2
- removed net TXBT: Q3.S, R18.2, U5.UARTTX
- removed net TX_5V: Q3.D, R19.2
- removed net USBVCC: Q1.D
- removed net VBATT: C2.1, IC7.EN, IC7.IN
- new net BT-RXI: U$3.1, U5.UARTRX
- new net BT-TXO: U$3.4, U5.UARTTX
- new net CHARGE: CN2.2, D1.C, S3.P, U$2.6
- new net N$10: U$2.1, U$2.4
- new net N$13: D11.A, R2.1
- new net PROG: R4.1, U2.PROG
- new net PROG-RXI: JP1.RXI, U$3.6
- new net PROG-TXO: JP1.TXO, U$3.3
- new net STAT: D11.C, U2.STAT
- net CTS: no longer R17.1, SJ4.2
- net DTR: now also JP1.DTR
- net GND: now also C3.2, CN1.1, JP1.GND, R4.2, U$2.3, U2.VSS, X1.GND; no longer C7.2, CN2.1, IC2A.V-, IC2B.+IN, IC2B.-IN, LED2.C, R5.1, SJ2.1, SJ3.1, U2.GND
- net N$1: now also C6.1, D1.A, U2.VBAT; no longer S3.P
- net N$2: now also CN2.1, U$2.2; no longer LED2.A, R2.1
- net N$8: now also CN1.2, U$2.5; no longer CN1.1, CN2.2
- net PWMA: now also U3.PD6(AIN0); no longer U3.PD3(INT1)
- net RTS: no longer Q2.S, R13.2, SJ4.1
- net RX-I: now also U$3.5
- net TX-O: now also U$3.2
- net VCC: now also C14.1, C18.1, C5.2, JP1.VCC, R10.2, R11.2, R3.2, SJ1.1, U$16.A, U$17.A, U$18.A, U1.VDD, U3.AVCC, U3.VCC@1, U3.VCC@2, U4.VCC, U5.VDD
- net VIN: now also C3.1, R2.2, U2.VIN, X1.VBUS; no longer R4.2
- net V_BATT: now also C17.1, C19.+, C2.1, IC7.EN, IC7.IN, U4.VM1, U4.VM2, U4.VM3
Other:
- note added: "Connection to 3.7V System"
- note added: "Set for 500mA charging"
- note added: "miniUSB"
- note removed: "**"
- note removed: "***"
- note removed: "3.3V 150mA Out"
- note removed: "3v3 Reg"
- note removed: "Comparator / 3.3V Regulator"
- moved on the sheet: C6, R2, R4

Commit message: Latest PIDDYBOT pcb finished ready to order
Parts:
- removed D1: (no value), SparkFun-DiscreteSemi:DIODESOD
- added D4: (no value), microbuilder:BAT54C
Connections:
- net CHARGE: now also D4.C; no longer D1.C
- net N$1: now also D4.A1, D4.A2; no longer D1.A
Changed lines of the file:
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@@
 <grid distance="0.1" unitdist="inch" unit="inch" style="lines" multiple="1" display="no" altdistance="0.01" altunitdist="inch" altunit="inch"/>
 <layers>
-<layer number="1" name="Top" color="4" fill="1" visible="yes" active="no"/>
-<layer number="16" name="Bottom" color="1" fill="1" visible="yes" active="no"/>
-<layer number="17" name="Pads" color="2" fill="1" visible="yes" active="no"/>
-<layer number="18" name="Vias" color="2" fill="1" visible="yes" active="no"/>
-<layer number="19" name="Unrouted" color="6" fill="1" visible="yes" active="no"/>
-<layer number="20" name="Dimension" color="15" fill="1" visible="yes" active="no"/>
-<layer number="21" name="tPlace" color="7" fill="1" visible="yes" active="no"/>
-<layer number="22" name="bPlace" color="7" fill="1" visible="yes" active="no"/>
-<layer number="23" name="tOrigins" color="15" fill="1" visible="yes" active="no"/>
-<layer number="24" name="bOrigins" color="15" fill="1" visible="yes" active="no"/>
-<layer number="25" name="tNames" color="7" fill="1" visible="yes" active="no"/>
-<layer number="26" name="bNames" color="7" fill="1" visible="yes" active="no"/>
-<layer number="27" name="tValues" color="7" fill="1" visible="yes" active="no"/>
-<layer number="28" name="bValues" color="7" fill="1" visible="yes" active="no"/>
+<layer number="1" name="Top" color="4" fill="1" visible="no" active="no"/>
+<layer number="16" name="Bottom" color="1" fill="1" visible="no" active="no"/>
+<layer number="17" name="Pads" color="2" fill="1" visible="no" active="no"/>
+<layer number="18" name="Vias" color="2" fill="1" visible="no" active="no"/>
+<layer number="19" name="Unrouted" color="6" fill="1" visible="no" active="no"/>
+<layer number="20" name="Dimension" color="15" fill="1" visible="no" active="no"/>
+<layer number="21" name="tPlace" color="7" fill="1" visible="no" active="no"/>
+<layer number="22" name="bPlace" color="7" fill="1" visible="no" active="no"/>
+<layer number="23" name="tOrigins" color="15" fill="1" visible="no" active="no"/>
+<layer number="24" name="bOrigins" color="15" fill="1" visible="no" active="no"/>
+<layer number="25" name="tNames" color="7" fill="1" visible="no" active="no"/>
+<layer number="26" name="bNames" color="7" fill="1" visible="no" active="no"/>
+<layer number="27" name="tValues" color="7" fill="1" visible="no" active="no"/>
+<layer number="28" name="bValues" color="7" fill="1" visible="no" active="no"/>
 <layer number="29" name="tStop" color="7" fill="3" visible="no" active="no"/>
 <layer number="30" name="bStop" color="7" fill="6" visible="no" active="no"/>
@@
 <layer number="35" name="tGlue" color="7" fill="4" visible="no" active="no"/>
 <layer number="36" name="bGlue" color="7" fill="5" visible="no" active="no"/>
-<layer number="37" name="tTest" color="7" fill="1" visible="yes" active="no"/>
-<layer number="38" name="bTest" color="7" fill="1" visible="yes" active="no"/>
+<layer number="37" name="tTest" color="7" fill="1" visible="no" active="no"/>
+<layer number="38" name="bTest" color="7" fill="1" visible="no" active="no"/>
 <layer number="39" name="tKeepout" color="4" fill="11" visible="no" active="no"/>
 <layer number="40" name="bKeepout" color="1" fill="11" visible="no" active="no"/>
@@
 <layer number="44" name="Drills" color="7" fill="1" visible="no" active="no"/>
 <layer number="45" name="Holes" color="7" fill="1" visible="no" active="no"/>
-<layer number="46" name="Milling" color="3" fill="1" visible="yes" active="no"/>
-<layer number="47" name="Measures" color="7" fill="1" visible="yes" active="no"/>
-<layer number="48" name="Document" color="7" fill="1" visible="yes" active="no"/>
-<layer number="49" name="Reference" color="7" fill="1" visible="yes" active="no"/>
-<layer number="50" name="dxf" color="7" fill="1" visible="yes" active="no"/>
-<layer number="51" name="tDocu" color="7" fill="1" visible="yes" active="no"/>
-<layer number="52" name="bDocu" color="7" fill="1" visible="yes" active="no"/>
-<layer number="53" name="tGND_GNDA" color="7" fill="9" visible="yes" active="no"/>
-<layer number="54" name="bGND_GNDA" color="1" fill="9" visible="yes" active="no"/>
-<layer number="56" name="wert" color="7" fill="1" visible="yes" active="no"/>
+<layer number="46" name="Milling" color="3" fill="1" visible="no" active="no"/>
+<layer number="47" name="Measures" color="7" fill="1" visible="no" active="no"/>
+<layer number="48" name="Document" color="7" fill="1" visible="no" active="no"/>
+<layer number="49" name="Reference" color="7" fill="1" visible="no" active="no"/>
+<layer number="50" name="dxf" color="7" fill="1" visible="no" active="no"/>
+<layer number="51" name="tDocu" color="7" fill="1" visible="no" active="no"/>
+<layer number="52" name="bDocu" color="7" fill="1" visible="no" active="no"/>
+<layer number="53" name="tGND_GNDA" color="7" fill="9" visible="no" active="no"/>
+<layer number="54" name="bGND_GNDA" color="1" fill="9" visible="no" active="no"/>
+<layer number="56" name="wert" color="7" fill="1" visible="no" active="no"/>
 <layer number="91" name="Nets" color="2" fill="1" visible="yes" active="yes"/>
 <layer number="92" name="Busses" color="1" fill="1" visible="yes" active="yes"/>
@@
 <part name="P+12" library="SparkFun" deviceset="VCC" device="" value="3.3V"/>
 <part name="P+13" library="SparkFun" deviceset="VCC" device="" value="3.3V"/>
-<part name="D1" library="SparkFun-DiscreteSemi" deviceset="DIODE" device="SOD"/>
+<part name="D4" library="microbuilder" deviceset="BAT54C" device=""/>
 </parts>
 <sheets>
 <sheet>
 <plain>
-<text x="205.74" y="147.32" size="2.54" layer="94" ratio="15">ATmega328</text>
+<text x="208.28" y="142.24" size="2.54" layer="94" ratio="15">ATmega328</text>
 <text x="466.598" y="72.898" size="1.778" layer="97">I2C Address Selection*</text>
 <text x="487.68" y="81.788" size="1.778" layer="97" rot="R180">*</text>
@@
 <instance part="P+12" gate="1" x="254" y="218.44"/>
 <instance part="P+13" gate="1" x="287.02" y="215.9"/>
-<instance part="D1" gate="G$1" x="177.8" y="-45.72"/>
+<instance part="D4" gate="G$1" x="177.8" y="-45.72"/>
 </instances>
 <busses>
@@
 </segment>
 <segment>
-<pinref part="D1" gate="G$1" pin="C"/>
 <wire x1="180.34" y1="-45.72" x2="187.96" y2="-45.72" width="0.1524" layer="91"/>
+<pinref part="D4" gate="G$1" pin="C"/>
+<label x="182.88" y="-45.72" size="1.778" layer="95"/>
 </segment>
 </net>
@@
 <pinref part="U2" gate="G$1" pin="VBAT"/>
 <pinref part="C6" gate="G$1" pin="1"/>
-<pinref part="D1" gate="G$1" pin="A"/>
-</segment>
-</net>
+<pinref part="D4" gate="G$1" pin="A2"/>
+<wire x1="175.26" y1="-45.72" x2="175.26" y2="-50.8" width="0.1524" layer="91"/>
+<wire x1="175.26" y1="-50.8" x2="177.8" y2="-50.8" width="0.1524" layer="91"/>
+<pinref part="D4" gate="G$1" pin="A1"/>
+<wire x1="175.26" y1="-45.72" x2="175.26" y2="-40.64" width="0.1524" layer="91"/>
+<wire x1="175.26" y1="-40.64" x2="177.8" y2="-40.64" width="0.1524" layer="91"/>
+<junction x="175.26" y="-45.72"/>
+</segment>
+</net>
