File: Board_V1_32U4/PIDDYBOT_V1.sch (EAGLE design)
At the start: 58 parts, among them CN2 M02JST-PTH-2, U1 MPU-6050-1, U2 MCP73831, U4 TB6621FNG, U5 BLUETOOTH-RN41, U6 MIC5219, Y1 8Mhz

Commit message: Changed power line for v_batt to v_motor
Connections:
- net V_BATT: no longer C15.+, D6.C, U6.EN, U6.IN
- net V_MOTOR: now also C15.+, D6.C, U6.EN, U6.IN
Changed lines of the file:
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@@
 <?xml version="1.0" encoding="utf-8"?>
 <!DOCTYPE eagle SYSTEM "eagle.dtd">
-<eagle version="6.5.0">
+<eagle version="7.1.0">
 <drawing>
 <settings>
@@
 </segment>
 <segment>
-<wire x1="236.22" y1="-53.34" x2="238.76" y2="-53.34" width="0.1524" layer="91"/>
-<wire x1="238.76" y1="-63.5" x2="236.22" y2="-63.5" width="0.1524" layer="91"/>
-<wire x1="236.22" y1="-63.5" x2="236.22" y2="-53.34" width="0.1524" layer="91"/>
-<wire x1="226.06" y1="-53.34" x2="236.22" y2="-53.34" width="0.1524" layer="91"/>
-<wire x1="226.06" y1="-55.88" x2="226.06" y2="-53.34" width="0.1524" layer="91"/>
-<wire x1="226.06" y1="-53.34" x2="226.06" y2="-48.26" width="0.1524" layer="91"/>
-<wire x1="226.06" y1="-48.26" x2="223.52" y2="-48.26" width="0.1524" layer="91"/>
-<junction x="236.22" y="-53.34"/>
-<junction x="226.06" y="-53.34"/>
-<pinref part="U6" gate="G$1" pin="IN"/>
-<pinref part="U6" gate="G$1" pin="EN"/>
-<pinref part="C15" gate="G$1" pin="+"/>
-<pinref part="D6" gate="G$1" pin="C"/>
-</segment>
-<segment>
 <pinref part="S2" gate="1" pin="P"/>
 <wire x1="40.64" y1="157.48" x2="30.48" y2="157.48" width="0.1524" layer="91"/>
@@
 <pinref part="S2" gate="1" pin="S"/>
 </segment>
-</net>
+<segment>
+<wire x1="236.22" y1="-53.34" x2="238.76" y2="-53.34" width="0.1524" layer="91"/>
+<wire x1="238.76" y1="-63.5" x2="236.22" y2="-63.5" width="0.1524" layer="91"/>
+<wire x1="236.22" y1="-63.5" x2="236.22" y2="-53.34" width="0.1524" layer="91"/>
+<wire x1="226.06" y1="-53.34" x2="236.22" y2="-53.34" width="0.1524" layer="91"/>
+<wire x1="226.06" y1="-55.88" x2="226.06" y2="-53.34" width="0.1524" layer="91"/>
+<wire x1="226.06" y1="-53.34" x2="226.06" y2="-48.26" width="0.1524" layer="91"/>
+<wire x1="226.06" y1="-48.26" x2="223.52" y2="-48.26" width="0.1524" layer="91"/>
+<junction x="236.22" y="-53.34"/>
+<junction x="226.06" y="-53.34"/>
+<pinref part="U6" gate="G$1" pin="IN"/>
+<pinref part="U6" gate="G$1" pin="EN"/>
+<pinref part="C15" gate="G$1" pin="+"/>
+<pinref part="D6" gate="G$1" pin="C"/>
+</segment>
+</net>

Commit message: latest PIDDYBOT 32u4 update
Parts:
- removed S2, S3: (no value), SparkFun-Electromechanical:SWITCH-SPDTPTH
- added C1: 1uF, SparkFun:CAP0603-CAP
- added L2: 33uH, SparkFun-Passives:INDUCTOR0402
- added LOGO1: IDLEHANDS_LOGOL, IdleHandsProject:IDLEHANDS_LOGOL
- added LOGO2: OSHW-LOGOM, SparkFun-Aesthetics:OSHW-LOGOM
- added R1: 1M, SparkFun:RESISTOR0603-RES
- added R3: 470k, SparkFun:RESISTOR0603-RES
- added S4: (no value), SparkFun-Electromechanical:SWITCH-SPDTPTH
Connections:
- removed net D11: U$1.PB7
- removed net N$4: D6.A, S3.S
- removed net VIO: C16.1, U1.VLOGIC
- removed net V_MOTOR: C15.+, C17.1, C19.+, D6.C, S2.S, U4.VM1, U4.VM2, U4.VM3, U6.EN, U6.IN
- new net BATT: C1.1, R1.1, R3.2
- new net ISOLATEDVCC: C14.1, C16.1, L2.2, U1.VDD, U1.VLOGIC
- new net RAW: C15.+, C17.1, C19.+, D6.C, R1.2, S4.P, U4.VM1, U4.VM2, U4.VM3, U6.EN, U6.IN
- net 3.3V: now also L2.1; no longer C14.1, U1.VDD
- net AIN1: now also U$1.PC6; no longer U$1.PC7
- net AIN2: now also U$1.PD6(ADC9); no longer U$1.PB6(ADC13)
- net GND: now also C1.2, R3.1, U1.CLKIN, U1.FSYNC
- net INT: now also U$1.PB7
- net MTE_A_2: now also U$1.PB6(ADC13); no longer U$1.PD6(ADC9)
- net N$3: now also D6.A; no longer S3.P
- net PWMB: now also U$1.PC7; no longer U$1.PC6
- net V_BATT: now also S4.O; no longer S2.P
Other:
- note removed: "Connection to 3.7V System"
- moved on the sheet: C14
